File: SMD PLACA.kicad_pcb (KiCad board)
At the start: 2 copper layers, 103.6 x 61.8 mm, 15 parts, among them J1 Screw_Terminal_01x02, J2 Screw_Terminal_01x05, J3 Screw_Terminal_01x02, J4 Screw_Terminal_01x04, J5 Screw_Terminal_01x04, Q2 IRL520, SW1 SW_SPST, U3 YAAJ_DCDC_StepDown_LM2596, U4 PC817

Commit message: 9/10
Parts:
- Q2: value IRL520 -> IRL520N
- moved RV1 9.32 mm to (130.2, 76.8)
Routing:
- net POT: track 35.3 -> 47.1 mm
- net +3.3V: track 60.9 -> 71.7 mm
- net +5V: track 48.9 -> 50.7 mm
- net +12V: track 70.8 -> 71.7 mm
Other:
- board text added: "10k"
- board text added: "33O"
- board text added: "ALIMENTACION"
- board text added: "R-C"
- board text added: "\"

Commit message: 13/10/2026
Parts:
- removed J4: Screw_Terminal_01x04, Connector_PinHeader_2.00mm:PinHeader_1x04_P2.00mm_Vertical
- added C1: 100uF, Capacitor_THT:C_Disc_D3.0mm_W1.6mm_P2.50mm, F.Cu at (117.5, 23.8)
- added H1: MountingHole, yamelxd:Ado-foto, F.Cu at (7.48, 9.16)
- added J6: Screw_Terminal_01x06, Connector_PinHeader_2.00mm:PinHeader_1x06_P2.00mm_Vertical, F.Cu at (131.0, 26.0)
- Q2: value IRL520N -> IRL520
- moved Q2 5.12 mm to (61.5, 34.9), turned to 0 degrees
Connections:
- J5 pad 1: SCL -> SDA
- J5 pad 2: SDA -> SCL
Routing:
- net VMOT: track 0.00 -> 27.0 mm
- net Net-(Q2-Pad1): track 24.7 -> 29.4 mm
- net GND: track 0.00 -> 3.72 mm
- net 1A: track 19.5 -> 20.5 mm
- net 2B: track 11.1 -> 12.1 mm
- net 2A: track 15.0 -> 16.0 mm
- net 1B: track 23.4 -> 24.4 mm
Other:
- board size 103.6 x 61.8 mm -> 103.6 x 62.6 mm
