File: SMD PLACA.kicad_sch (KiCad schematic)
At the start: 15 parts, among them J1 Screw_Terminal_01x02, J2 Screw_Terminal_01x05, J3 Screw_Terminal_01x02, J4 Screw_Terminal_01x04, J5 Screw_Terminal_01x04, Q2 IRL520, SW1 SW_SPST, U3 YAAJ_DCDC_StepDown_LM2596, U4 PC817

Commit message: 13/10/2026
Parts:
- removed J4: Screw_Terminal_01x04, Connector_PinHeader_2.00mm:PinHeader_1x04_P2.00mm_Vertical, symbol Connector:Screw_Terminal_01x04
- added C1: 100uF, Capacitor_THT:C_Disc_D3.0mm_W1.6mm_P2.50mm, symbol Device:C
- added H1: MountingHole, symbol Mechanical:MountingHole
- added J6: Screw_Terminal_01x06, Connector_PinHeader_2.00mm:PinHeader_1x06_P2.00mm_Vertical, symbol Connector:Screw_Terminal_01x06
Connections:
- net 1A: now also J6.3 (Pin_3)
- net 1B: now also J6.4 (Pin_4)
- net 2A: now also J6.2 (Pin_2)
- net 2B: now also J6.1 (Pin_1)
- net GND: now also C1.2, J6.6 (Pin_6)
- net VMOT: now also C1.1, J6.5 (Pin_5)
